Commit message: Completed till DWAPlanner.

File: abot_description/urdf/robot.gazebo.xacro (robot description, xacro)
@@ -25,4 +25,10 @@
         <material>Gazebo/FlatBlack</material>
     </gazebo>
+  <gazebo reference="imu_link">
+    <sensor type="imu" name="imu">
+      <always_on>true</always_on>
+    </sensor>
+    <material>Gazebo/FlatBlack</material>
+  </gazebo>
     <gazebo>
         <plugin name="abot_controller" filename="libgazebo_ros_diff_drive.so">
@@ -33,5 +39,5 @@
         <publishOdomTF>true</publishOdomTF>
         <robotBaseFrame>base_link</robotBaseFrame>
-        <publishWheelTF>true</publishWheelTF>
+        <publishWheelTF>false</publishWheelTF>
         <publishTf>true</publishTf>
         <publishWheelJointState>true</publishWheelJointState>
@@ -43,14 +49,8 @@
         <wheelDiameter>0.050</wheelDiameter>
         <wheelAcceleration>1</wheelAcceleration>
-        <wheelTorque>20</wheelTorque>
+        <wheelTorque>10</wheelTorque>
         <rosDebugLevel>na</rosDebugLevel>
         </plugin>
     </gazebo>
-  <gazebo reference="imu_link">
-    <sensor type="imu" name="imu">
-      <always_on>true</always_on>
-    </sensor>
-    <material>Gazebo/FlatBlack</material>
-  </gazebo>
   <gazebo>
     <plugin name="imu_plugin" filename="libgazebo_ros_imu.so">
@@ -85,4 +85,5 @@
     <sensor type="ray" name="lds_lfcd_sensor">
       <pose>0 0 0 0 0 0</pose>
+      <visualize>false</visualize>
       <update_rate>5</update_rate>
       <ray>

File: abot_description/urdf/robot.urdf.xacro (robot description, xacro)
@@ -6,5 +6,5 @@
 <parent link="base_link"/>
 <child link="chassis" />
-<origin rpy="0.0 0 0" xyz="0 0 0"/>
+<origin  xyz="0 0 0.005" rpy="0 0 -1.5708"/>
 </joint>
 <link name="chassis">
@@ -51,5 +51,5 @@
 </collision>
 <inertial>
-<origin xyz="0 2.01808e-18 -0.009" rpy="0 0 0"/>
+<origin xyz="0 2.01808e-18 -0.009" rpy="-1.5708 0 0"/>
 <mass value="1.26704" />
 <inertia ixx="0.000232186" ixy="0"  ixz="0" iyy="0.000395951" iyz="0" izz="0.000232186" />
@@ -61,6 +61,4 @@
 <child link="wheel" />
 <axis xyz="0 0 -1"/>
-<limit effort="1" velocity="20"/>
-<joint_properties friction="0.0"/>
 </joint>
 <!-- Transmission is important to link the joints and the controller -->
@@ -93,5 +91,5 @@
 </collision>
 <inertial>
-<origin xyz="0 -2.01808e-18 -0.009" rpy="0 0 0"/>
+<origin xyz="0 -2.01808e-18 -0.009" rpy="-1.5708 0 0"/>
 <mass value="1.26704" />
 <inertia ixx="0.000232186" ixy="0"  ixz="0" iyy="0.000395951" iyz="0" izz="0.000232186" />
@@ -103,6 +101,4 @@
 <child link="wheel_2" />
 <axis xyz="0 0 1"/>
-<limit effort="1" velocity="20" />
-<joint_properties friction="0.0"/>
 </joint>
 <!-- Transmission is important to link the joints and the controller -->
@@ -145,17 +141,18 @@
 <child link="roller" />
 <axis xyz="0 0 1"/>
-<joint_properties friction="0.0"/>
 </joint>
 <!--Lidar and imu -->
   <joint name="imu_joint" type="fixed">
-    <parent link="base_link"/>
+    <parent link="chassis"/>
     <child link="imu_link"/>
-    <origin xyz="0 0 0" rpy="0 0 0"/>
+    <!--<origin xyz="-0.032 0 0.068" rpy="0 0 0"/>-->
+    <origin xyz="0 0 0" rpy="0 0 0"/>-->
   </joint>
   <link name="imu_link"/>
   <joint name="scan_joint" type="fixed">
-    <parent link="base_link"/>
+    <parent link="chassis"/>
     <child link="base_scan"/>
-    <origin xyz="0 0 0.096" rpy="0 0 -1.57"/>
+    <!--<origin xyz="-0.032 0 0.172" rpy="0 0 0"/>-->
+    <origin xyz="0 0 0.096" rpy="0 0 -1.5708"/>
   </joint>
   <link name="base_scan">
