Commit message: Added Intel Realsense D435

File: abot_description/urdf/robot.urdf.xacro (robot description, xacro)
@@ -2,4 +2,5 @@
 <robot name="abot" xmlns:xacro="http://ros.org/wiki/xacro">
 <xacro:include filename="$(find abot_description)/urdf/robot.gazebo.xacro"/>
+<xacro:include filename="$(find abot_description)/urdf/_d435.urdf.xacro" />
 <link name="base_link"></link>
 <joint name="base_link_to_base" type="fixed">
@@ -12,5 +13,5 @@
 <origin xyz="9.21702e-10 0.00447478 0.0341544" rpy="0 -0 0" />
 <geometry>
-<mesh filename="package://abot_description/urdf/chassis.stl"/>
+<mesh filename="package://abot_description/meshes/chassis.stl"/>
 </geometry>
 <material name="chassis_material">
@@ -21,5 +22,5 @@
 <origin xyz="9.21702e-10 0.00447478 0.0341544" rpy="0 -0 0" />
 <geometry>
-<mesh filename="package://abot_description/urdf/chassis.stl"/>
+<mesh filename="package://abot_description/meshes/chassis.stl"/>
 </geometry>
 <material name="chassis_material">
@@ -37,5 +38,5 @@
 <origin xyz="0 0 -0.009" rpy="-1.5708 -1.5708 0" />
 <geometry>
-<mesh filename="package://abot_description/urdf/wheel.stl"/>
+<mesh filename="package://abot_description/meshes/wheel.stl"/>
 </geometry>
 <material name="wheel_material">
@@ -77,5 +78,5 @@
 <origin xyz="0 0 -0.009" rpy="1.5708 1.5708 0" />
 <geometry>
-<mesh filename="package://abot_description/urdf/wheel.stl"/>
+<mesh filename="package://abot_description/meshes/wheel.stl"/>
 </geometry>
 <material name="wheel_material">
@@ -117,5 +118,5 @@
 <origin xyz="0 0 -0.094554" rpy="-1.5708 -1.5708 0" />
 <geometry>
-<mesh filename="package://abot_description/urdf/roller.stl"/>
+<mesh filename="package://abot_description/meshes/roller.stl"/>
 </geometry>
 <material name="roller_material">
@@ -160,5 +161,5 @@
       <origin xyz="0 0 0.0" rpy="0 0 0"/>
       <geometry>
-        <mesh filename="package://abot_description/urdf/lds.stl" scale="0.001 0.001 0.001"/>
+        <mesh filename="package://abot_description/meshes/lds.stl" scale="0.001 0.001 0.001"/>
       </geometry>
       <material name="dark"/>
@@ -178,3 +179,6 @@
     </inertial>
   </link>
+  <xacro:sensor_d435 name="camera" topics_ns="camera" parent="chassis" publish_pointcloud="true">
+    <origin xyz="0 0.08 0.065" rpy="0 -0.139626 1.5708" /> <!-- tilted 8 degree up -->
+  </xacro:sensor_d435>
 </robot>
